File: hardware/ethernet.kicad_sch (KiCad schematic)
At the start: 39 parts, among them J1 RJ45_Hanrun_HR911105A_Horizon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, U1 W5500, Y1 25MHz

Commit message: Added Board Register
Parts:
- removed C1, C6: 1uF, Capacitor_SMD:C_0603_1608Metric, symbol Device:C_Small
- removed C11, C12, C13, C16, C4, C5, C7, C9: 100nF, Capacitor_SMD:C_0603_1608Metric, symbol Device:C_Small
- removed L1: 120R @ 100MHz, Inductor_SMD:L_0603_1608Metric, symbol Device:L_Ferrite_Small
- removed TP1: TestPoint_Small, TestPoint:TestPoint_Pad_D1.5mm, symbol Connector:TestPoint_Small
Other:
- moved on the sheet: C10, C14, C15, C17, C18, C19, C2, C3, C8, J1, R1, R10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

Commit message: Fixed some erros, changed to 3V
Parts:
- removed U1: W5500, Package_QFP:LQFP-48_7x7mm_P0.5mm, symbol Interface_Ethernet:W5500
- added U9: W5500, Package_QFP:LQFP-48_7x7mm_P0.5mm, symbol Interface_Ethernet:W5500
- renumbered J1 to J4, Y1 to Y3
Connections:
- net +3.3V: now also U9.28 (VDD), U9.43 (PMODE2), U9.44 (PMODE1), U9.45 (PMODE0)
- net +3.3VA: now also U9.11 (AVDD), U9.15 (AVDD), U9.17 (AVDD), U9.21 (AVDD), U9.4 (AVDD), U9.8 (AVDD)
- net ACT_LED: now also U9.27 (ACTLED)
- net GND: now also U9.14 (AGND), U9.16 (AGND), U9.19 (AGND), U9.29 (GND), U9.3 (AGND), U9.48 (AGND), U9.9 (AGND)
- net RXN: now also U9.5 (RXN)
- net RXP: now also U9.6 (RXP)
- net TXN: now also U9.1 (TXN)
- net TXP: now also U9.2 (TXP)
- net W5500_LINK: now also U9.25 (LINKLED)
- net at C8.1: now also U9.22 (1V2O)
- net at C3.2, Y3.1: now also U9.31 (XO)
- net at C2.2, Y3.3: now also U9.30 (XI/CLKIN)
- net at R6.1: now also U9.10 (EXRES1)
- net at C10.1: now also U9.20 (TOCAP)
- net W5500_CS renamed SPI_CS_{1}
- net SPI_CS_{1}: now also U9.32 (~{SCS})
- net W5500_INT renamed INTERNAL_IRQ
- net INTERNAL_IRQ: now also U9.36 (~{INT})
- net W5500_RST renamed MR
- net MR: now also U9.37 (~{RST})
- new net MISO: U9.34 (MISO)
- new net MOSI: U9.35 (MOSI)
- new net SCK: U9.33 (SCLK)
