File: hardware/video.kicad_sch (KiCad schematic)
At the start: 11 parts, among them J6 DE15_Socket_HighDensity, U13 V9958, U14 74AUC2G32, U15 41464, U16 41464, U17 41464, U18 41464, U19 SN74LVC245APW, U21 LM1881, U22 74LVC1G07, Y3 TFT680

Commit message: Minor Improvemnts
Parts:
- J6: footprint (none) -> Connector_Dsub:DSUB-15_Socket_Horizontal_P2.77x2.84mm_EdgePinOffset9.40mm
- U14: footprint (none) -> Package_SO:SSOP-8_2.95x2.8mm_P0.65mm
- U15, U16, U17, U18: footprint (none) -> Package_DIP:DIP-18_W7.62mm
- U21: footprint (none) -> Package_DIP:DIP-8_W7.62mm
- U22: footprint (none) -> Package_TO_SOT_SMD:SOT-23-5

Commit message: Add new categories for Video&Audio and Sound System in project configuration
Parts:
- removed unit 1 of U14
- removed unit 2 of U14
- removed U19: SN74LVC245APW, Package_SO:TSSOP-20_4.4x6.5mm_P0.65mm, symbol Logic_LevelTranslator:SN74LVC245APW
- renumbered U22 to U15, U13 to U17, U21 to U18, U15 to U19, U16 to U21, U17 to U22, U18 to U23, Y3 to Y2
Connections:
- net MR: no longer U17.9 (~{RESET})
- net ~{CSW}: now reaches U17.30 (~{CSW})
- net D5V7: now reaches U17.32 (D7)
- net D5V6: now reaches U17.34 (D6)
- net D5V5: now reaches U17.35 (D5)
- net D5V4: now reaches U17.36 (D4)
- net D5V3: now reaches U17.37 (D3)
- net D5V2: now reaches U17.38 (D2)
- net D5V1: now reaches U17.39 (D1)
- net D5V0: now reaches U17.40 (D0)
- net ~{CSR}: now reaches U17.31 (~{CSR})
- new net ~{RESET}: U17.9 (~{RESET})

Commit message: Moved connection to external connections
Parts:
- removed J6: DE15_Socket_HighDensity, Connector_Dsub:DSUB-15_Socket_Horizontal_P2.77x2.84mm_EdgePinOffset9.40mm, symbol Connector:DE15_Socket_HighDensity
- removed U14: 74AUC2G32, Package_SO:SSOP-8_2.95x2.8mm_P0.65mm, symbol 74xGxx:74AUC2G32
Connections:
- net MR is gone; now on net ~{RESET}: U18.6 (RSET)
- net VSYNC: now reaches U18.3 (VSOUT)
- no-connect marks 25 -> 20
Other:
- moved on the sheet: U18

Commit message: PCD DESIGN
Parts:
- VPU1: renamed from U17; footprint (none) -> footprints:SDIP-64_V9958
- renumbered U21 to RAM_H1, U23 to RAM_H2, U19 to RAM_L1, U22 to RAM_L2
Other:
- moved on the sheet: U18
Changed lines of the file:
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@@
 	)
 	(no_connect
-		(at 187.96 140.97)
+		(at 148.59 132.08)
 	)
 	(no_connect
@@
 	)
 	(no_connect
-		(at 187.96 148.59)
+		(at 148.59 139.7)
 	)
 	(no_connect
@@
 	)
 	(no_connect
-		(at 187.96 146.05)
+		(at 148.59 137.16)
 	)
 	(bus_entry
@@
 	)
 	(label "CSYNC"
-		(at 213.36 143.51 0)
+		(at 173.99 134.62 0)
 		(effects
 			(font
@@
 	(global_label "VSYNC"
 		(shape output)
-		(at 187.96 143.51 180)
+		(at 148.59 134.62 180)
 		(fields_autoplaced yes)
 		(effects
@@
 		)
 		(property "Intersheetrefs" "${INTERSHEET_REFS}"
-			(at 178.5116 143.51 0)
+			(at 139.1416 134.62 0)
 			(effects
 				(font
@@
 	(hierarchical_label "~{RESET}"
 		(shape input)
-		(at 213.36 148.59 0)
+		(at 173.99 139.7 0)
 		(effects
 			(font
@@
 		(on_board yes)
 		(dnp no)
-		(property "Reference" "U22"
+		(property "Reference" "RAM_L2"
 			(at 237.744 27.686 0)
 			(effects
@@
 			(project "Lambda One"
 				(path "/73ea9964-373f-4fdc-b03e-f532cf836c0d/17c7449d-caad-4fd1-a972-8af3d0bf5f54/de4b84de-a9b1-46be-baf2-2295df779266"
-					(reference "U22")
+					(reference "RAM_L2")
 					(unit 1)
 				)
@@
 		(on_board yes)
 		(dnp no)
-		(property "Reference" "U23"
+		(property "Reference" "RAM_H2"
 			(at 237.744 70.866 0)
 			(effects
@@
 			(project "Lambda One"
 				(path "/73ea9964-373f-4fdc-b03e-f532cf836c0d/17c7449d-caad-4fd1-a972-8af3d0bf5f54/de4b84de-a9b1-46be-baf2-2295df779266"
-					(reference "U23")
+					(reference "RAM_H2")
 					(unit 1)
 				)
@@
 	(symbol
 		(lib_id "Video:LM1881")
-		(at 200.66 146.05 0)
+		(at 161.29 137.16 0)
 		(mirror y)
 		(unit 1)
@@
 		(dnp no)
 		(property "Reference" "U18"
-			(at 203.7781 156.21 0)
+			(at 164.4081 147.32 0)
 			(effects
 				(font
@@
 		)
 		(property "Value" "LM1881"
-			(at 203.7781 153.67 0)
+			(at 164.4081 144.78 0)
 			(effects
 				(font
@@
 		)
 		(property "Footprint" "Package_DIP:DIP-8_W7.62mm"
-			(at 200.66 162.052 0)
+			(at 161.29 153.162 0)
 			(effects
 				(font
@@
 		)
 		(property "Datasheet" "https://www.ti.com/lit/ds/symlink/lm1881.pdf"
-			(at 200.66 159.766 0)
+			(at 161.29 150.876 0)
 			(effects
 				(font
@@
 		)
 		(property "Description" "Video Sync Separator, composite sync and vertical sync outputs, DIP-8 / SOIC-8"
-			(at 200.66 157.48 0)
+			(at 161.29 148.59 0)
 			(effects
 				(font
@@
 		(on_board yes)
 		(dnp no)
-		(property "Reference" "U21"
+		(property "Reference" "RAM_H1"
 			(at 184.404 70.866 0)
 			(effects
@@
 			(project "Lambda One"
 				(path "/73ea9964-373f-4fdc-b03e-f532cf836c0d/17c7449d-caad-4fd1-a972-8af3d0bf5f54/de4b84de-a9b1-46be-baf2-2295df779266"
-					(reference "U21")
+					(reference "RAM_H1")
 					(unit 1)
 				)
@@
 	(symbol
 		(lib_id "power:+5V")
-		(at 200.66 135.89 0)
+		(at 161.29 127 0)
 		(unit 1)
 		(exclude_from_sim no)
@@
 		(dnp no)
 		(property "Reference" "#PWR091"
-			(at 200.66 139.7 0)
+			(at 161.29 130.81 0)
 			(effects
 				(font
@@
 		)
 		(property "Value" "+5V"
-			(at 200.66 132.08 0)
+			(at 161.29 123.19 0)
 			(effects
 				(font
@@
 		)
 		(property "Footprint" ""
-			(at 200.66 135.89 0)
+			(at 161.29 127 0)
 			(effects
 				(font
@@
 		)
 		(property "Datasheet" ""
-			(at 200.66 135.89 0)
+			(at 161.29 127 0)
 			(effects
 				(font
@@
 		)
 		(property "Description" "Power symbol creates a global label with name \"+5V\""
-			(at 200.66 135.89 0)
+			(at 161.29 127 0)
 			(effects
 				(font
@@
 		(on_board yes)
 		(dnp no)
-		(property "Reference" "U19"
+		(property "Reference" "RAM_L1"
 			(at 184.404 27.686 0)
 			(effects
@@
 			(project "Lambda One"
 				(path "/73ea9964-373f-4fdc-b03e-f532cf836c0d/17c7449d-caad-4fd1-a972-8af3d0bf5f54/de4b84de-a9b1-46be-baf2-2295df779266"
-					(reference "U19")
+					(reference "RAM_L1")
 					(unit 1)
 				)
@@
 		(on_board yes)
 		(dnp no)
-		(property "Reference" "U17"
+		(property "Reference" "VPU1"
 			(at 112.522 27.94 0)
 			(effects
@@
 			)
 		)
-		(property "Footprint" ""
+		(property "Footprint" "footprints:SDIP-64_V9958"
 			(at 119.38 53.34 0)
 			(effects
@@
 			(project "Lambda One"
 				(path "/73ea9964-373f-4fdc-b03e-f532cf836c0d/17c7449d-caad-4fd1-a972-8af3d0bf5f54/de4b84de-a9b1-46be-baf2-2295df779266"
-					(reference "U17")
+					(reference "VPU1")
 					(unit 1)
 				)
@@
 	(symbol
 		(lib_id "power:GND")
-		(at 200.66 153.67 0)
+		(at 161.29 144.78 0)
 		(unit 1)
 		(exclude_from_sim no)
@@
 		(fields_autoplaced yes)
 		(property "Reference" "#PWR092"
-			(at 200.66 160.02 0)
+			(at 161.29 151.13 0)
 			(effects
 				(font
@@
 		)
 		(property "Value" "GND"
-			(at 200.66 158.75 0)
+			(at 161.29 149.86 0)
 			(effects
 				(font
@@
 		)
 		(property "Footprint" ""
-			(at 200.66 153.67 0)
+			(at 161.29 144.78 0)
 			(effects
 				(font
@@
 		)
 		(property "Datasheet" ""
-			(at 200.66 153.67 0)
+			(at 161.29 144.78 0)
 			(effects
 				(font
@@
 		)
 		(property "Description" "Power symbol creates a global label with name \"GND\" , ground"
-			(at 200.66 153.67 0)
+			(at 161.29 144.78 0)
 			(effects
 				(font
