File: hardware/serial.kicad_sch (KiCad schematic)
At the start: 9 parts, among them J5 USB_C_Receptacle_USB2.0_14P, J7 USB_A, U10 CH340C, U20 CH340C, U5 SC16C654DBIB64_151

Commit message: PCD DESIGN
Parts:
- J7: footprint (none) -> Connector_USB:USB_A_Molex_67643_Horizontal
- renumbered U5 to SERIAL1, U20 to UART_USBA1, U10 to UART_USBC1
Changed lines of the file:
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@@
 		(on_board yes)
 		(dnp no)
-		(fields_autoplaced yes)
-		(property "Reference" "U10"
-			(at 185.9981 86.36 0)
+		(property "Reference" "UART_USBC1"
+			(at 169.164 86.36 0)
 			(effects
 				(font
@@
 		)
 		(property "Value" "CH340C"
-			(at 185.9981 88.9 0)
+			(at 184.15 86.614 0)
 			(effects
 				(font
@@
 			(project "Lambda One"
 				(path "/73ea9964-373f-4fdc-b03e-f532cf836c0d/ddbbde09-39b7-4f71-b314-84c8e93fa330"
-					(reference "U10")
+					(reference "UART_USBC1")
 					(unit 1)
 				)
@@
 		(dnp no)
 		(fields_autoplaced yes)
-		(property "Reference" "U5"
-			(at 104.14 74.422 0)
+		(property "Reference" "SERIAL1"
+			(at 108.8233 45.72 0)
 			(effects
 				(font
 					(size 1.524 1.524)
 				)
+				(justify left)
 			)
 		)
 		(property "Value" "SC16C654DBIB64_151"
-			(at 103.886 94.996 90)
+			(at 108.8233 48.26 0)
 			(effects
 				(font
 					(size 1.524 1.524)
 				)
+				(justify left)
 			)
 		)
@@
 			(project "Lambda One"
 				(path "/73ea9964-373f-4fdc-b03e-f532cf836c0d/ddbbde09-39b7-4f71-b314-84c8e93fa330"
-					(reference "U5")
+					(reference "SERIAL1")
 					(unit 1)
 				)
@@
 		(dnp no)
 		(fields_autoplaced yes)
-		(property "Reference" "U20"
+		(property "Reference" "UART_USBA1"
 			(at 184.7281 135.89 0)
 			(effects
@@
 			(project "Lambda One"
 				(path "/73ea9964-373f-4fdc-b03e-f532cf836c0d/ddbbde09-39b7-4f71-b314-84c8e93fa330"
-					(reference "U20")
+					(reference "UART_USBA1")
 					(unit 1)
 				)
@@
 		(dnp no)
 		(fields_autoplaced yes)
-		(property "Reference" "U5"
+		(property "Reference" "SERIAL1"
 			(at 35.56 145.542 0)
 			(effects
@@
 			(project "Lambda One"
 				(path "/73ea9964-373f-4fdc-b03e-f532cf836c0d/ddbbde09-39b7-4f71-b314-84c8e93fa330"
-					(reference "U5")
+					(reference "SERIAL1")
 					(unit 2)
 				)
@@
 			)
 		)
-		(property "Footprint" ""
+		(property "Footprint" "Connector_USB:USB_A_Molex_67643_Horizontal"
 			(at 212.09 119.38 0)
 			(effects

Commit message: Removed old VPU
Parts:
- added C18, C35: 47uF, Capacitor_SMD:C_0603_1608Metric, symbol Device:C_Small
- added C32, C33: 30pF, Capacitor_SMD:C_0603_1608Metric, symbol Device:C_Small
- added Y2: Crystal, Crystal:Crystal_HC49-U_Vertical, symbol Device:Crystal
- SERIAL1: footprint Package_QFP:LQFP-64_7x7mm_P0.4mm -> Package_LCC:PLCC-68
Connections:
- net +3.3V: now also UART_USBA1.16 (VCC), UART_USBC1.16 (VCC), C18.1, C35.1
- net GND: now also C18.2, C32.2, C33.2, C35.2
- net at SERIAL1.36 (XTAL2): now also C33.1, Y2.2
- net CLK: no longer names the net of SERIAL1.35 (XTAL1)
- net CLK: now also C32.1, Y2.1
- net VBUS_{1}: no longer names the net of J5.A4 (VBUS), J5.A9 (VBUS), J5.B4 (VBUS), J5.B9 (VBUS)
- net VBUS_{1}: no longer UART_USBC1.16 (VCC)
- net VBUS_{2}: no longer names the net of J7.1 (VBUS)
- net VBUS_{2}: no longer UART_USBA1.16 (VCC)
- no-connect marks 17 -> 18
