File: hardware/Lambda One.kicad_pcb (KiCad board)
At the start: 4 copper layers, 250 x 150 mm, 95 parts, among them IC1 DS1818, J1 Conn_01x02, J11 Conn_01x02, J12 Conn_01x02, J5 USB_C_Receptacle_USB2.0_14P, J7 USB_A, SW1 SW_Push, U14 74AUC2G32, U15 74LVC1G07, U18 LM1881, U25 SN74LVC8T245, U26 SN74LVC2T45DCUR, U27 SN74LVC1T45DBV, U28 74AHC1G08, U6 74HC00, U8 74HC00, U9 74HC00, Y1 TFT680, Y2 TFT680

Commit message: Las c with VPU
Parts:
- moved J11 234.7 mm to (22.8, 31.8)
- moved J12 234.7 mm to (22.8, 41.8)
- moved C8 74.0 mm to (94.7, 97.0)
- moved C12 55.5 mm to (94.7, 90.5)
- moved C15 54.0 mm to (94.5, 87.5)
- moved C17 47.0 mm to (94.8, 93.5)
- moved C14 29.1 mm to (68.7, 111.5), turned to 180 degrees
- moved L1 22.2 mm to (94.5, 84.5)
Routing:
- net AUDIO_{VDD}: track 253.4 -> 47.6 mm
- net +5VA: track 205.9 -> 26.3 mm, vias 8 -> 2
- net GND: track 360.3 -> 307.2 mm, vias 22 -> 20
- net +5V: track 468.7 -> 458.7 mm, vias 19 -> 15
- net (no net): track 0.00 -> 2.49 mm, vias 26 -> 23
- net RED: track 79.3 -> 77.2 mm
- net Net-(AUDIO_AMPL1-L): track 9.56 -> 8.70 mm, vias 1 -> 0
- net MR: vias 9 -> 7

Commit message: Removed old VPU
Parts:
- removed AUDIO_AMPL1: pam8403, pam8403:pam8403
- removed C16, C17: 100nF, Capacitor_SMD:C_0603_1608Metric
- removed C18, C19: 22nF, Capacitor_SMD:C_0603_1608Metric
- removed C22: 470pF, Capacitor_SMD:C_0603_1608Metric
- removed C24: 10µF, Capacitor_SMD:C_0603_1608Metric
- removed DB5V1: SN74LVC245AN, Package_DIP:DIP-20_W7.62mm
- removed L1: 120R @ 100MHz, Inductor_SMD:L_0603_1608Metric
- removed R5: 1k, Resistor_SMD:R_0603_1608Metric
- removed R6: 10k, Resistor_SMD:R_0603_1608Metric
- removed RAM_H1, RAM_H2, RAM_L1, RAM_L2: 41464, Package_DIP:DIP-18_W7.62mm
- removed SID1: SID, Package_DIP:DIP-28_W15.24mm_Socket
- removed SPI_EXT_{3}2: Conn_02x07_Odd_Even, Connector_PinSocket_2.54mm:PinSocket_2x07_P2.54mm_Vertical
- removed TP1: TestPoint_Small, TestPoint:TestPoint_Pad_D1.5mm
- removed U14: 74AUC2G32, Package_SO:SSOP-8_2.95x2.8mm_P0.65mm
- removed U15: 74LVC1G07, Package_TO_SOT_SMD:SOT-23-5
- removed U18: LM1881, Package_DIP:DIP-8_W7.62mm
- removed U26: SN74LVC2T45DCUR, Package_SO:VSSOP-8_2.3x2mm_P0.5mm
- removed VGA1: DE15_Socket_HighDensity, Connector_Dsub:DSUB-15_Socket_Horizontal_P2.77x2.84mm_EdgePinOffset9.40mm
- removed VPU1: V9958, footprints:SDIP-64_V9958
- removed Y2: TFT680, Oscillator:Oscillator_DIP-14
- added AUDIO_AMPL2: pam8403, pam8403:pam8403, F.Cu at (181.6, 37.8)
- added R7: 1k, Resistor_SMD:R_0603_1608Metric, F.Cu at (193.0, 45.9)
- added R8: 10k, Resistor_SMD:R_0603_1608Metric, F.Cu at (193.0, 48.4)
- added SID2: SID, Package_DIP:DIP-28_W15.24mm_Socket, F.Cu at (154.8, 29.2)
- added U1: SN74LVC8T245, Package_SO:SSOP-24_3.9x8.7mm_P0.635mm, F.Cu at (176.1, 54.9)
- added U2: 2.42OLED, old:DIYMORE.CC, F.Cu at (34.7, 70.0)
- C12: value 100nF -> 470pF
- C15: value 100nF -> 10µF
- C3: value 1uF -> 22nF
- C8: value 100nF -> 22nF
- SERIAL1: footprint Package_QFP:LQFP-64_7x7mm_P0.4mm -> Package_LCC:PLCC-68
- U25: footprint Package_DIP:DIP-20_W7.62mm -> Package_SO:SSOP-24_3.9x8.7mm_P0.635mm
- moved CPU1 209.1 mm to (35.5, 105.9)
- moved C2 203.9 mm to (83.0, 141.2), turned to 0 degrees
- moved C4 176.7 mm to (83.0, 143.7), turned to 0 degrees
- moved C5 174.6 mm to (83.0, 146.2), turned to 0 degrees
- moved ADDR1 168.3 mm to (53.9, 105.9)
- moved R3 168.1 mm to (91.0, 138.7), turned to 0 degrees
- moved R17 165.5 mm to (91.0, 143.7)
- moved U9 164.9 mm to (75.5, 120.2)
- moved C7 163.8 mm to (83.0, 151.2)
- moved Y1 163.5 mm to (66.6, 114.8), turned to 0 degrees
- moved C11 163.3 mm to (87.0, 141.2), turned to 0 degrees
- moved R16 162.0 mm to (91.0, 141.2)
- moved C1 159.2 mm to (83.0, 138.7)
- moved CPU_DB1 155.5 mm to (53.9, 137.9)
- moved C9 153.8 mm to (87.0, 138.7)
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Connections:
- C12 pad 1: +5VA -> Net-(SID2-POT_X)
- C15 pad 1: +5VA -> Net-(SID2-AUDIO_OUT)
- C15 pad 2: GND -> Net-(C15-Pad2)
- C3 pad 1: +5VA -> Net-(SID2-CAP_1A)
- C3 pad 2: GND -> Net-(SID2-CAP_1B)
- C8 pad 1: +5VA -> Net-(SID2-CAP_2A)
- C8 pad 2: GND -> Net-(SID2-CAP_2B)
- SPI_EXT_{3}1 pad 12: SPI_CS_{3} -> SPI_CS_{4}
- U25 pad 14: /Video&Audio/Sound System/Addr5V4 -> /Audio/Addr5V4
- U25 pad 15: /Video&Audio/Sound System/Addr5V3 -> /Audio/Addr5V3
- U25 pad 16: /Video&Audio/Sound System/Addr5V2 -> /Audio/Addr5V2
- U25 pad 17: /Video&Audio/Sound System/Addr5V1 -> /Audio/Addr5V1
- U25 pad 18: /Video&Audio/Sound System/Addr5V0 -> /Audio/Addr5V0
- U25 pad 19: /Video&Audio/Sound System/~{CS} -> Net-(SID2-~{CS})
- U25 pad 20: /Video&Audio/Sound System/R/~{W} -> Net-(SID2-R/~{W})
- U27 pad 4: /Video&Audio/Sound System/~{RESET} -> Net-(SID2-~{RES})
- U28 pad 4: /Video&Audio/~{OE} -> /Audio/~{OE}
Routing:
- net +3.3V: track 1066.6 -> 0.00 mm, vias 80 -> 0
- net +5V: track 458.7 -> 0.00 mm, vias 15 -> 0
- net CLK: track 453.3 -> 0.00 mm, vias 26 -> 0
- net Addr3: track 449.4 -> 0.00 mm, vias 17 -> 0
- net Addr1: track 425.3 -> 0.00 mm, vias 23 -> 0
- net ~{IRQ}: track 375.5 -> 0.00 mm, vias 11 -> 0
- net D7: track 357.8 -> 0.00 mm, vias 22 -> 0
- net D3: track 352.1 -> 0.00 mm, vias 18 -> 0
- net D5: track 341.7 -> 0.00 mm, vias 13 -> 0
- net D6: track 330.5 -> 0.00 mm, vias 18 -> 0
- net D0: track 314.4 -> 0.00 mm, vias 12 -> 0
- net D1: track 310.8 -> 0.00 mm, vias 16 -> 0
- net D4: track 310.4 -> 0.00 mm, vias 14 -> 0
- net Addr0: track 310.3 -> 0.00 mm, vias 22 -> 0
- net MR: track 308.7 -> 0.00 mm, vias 7 -> 0
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- removed copper zone on In1.Cu, net GND
Other:
- board outline removed

Commit message: Minor changes
Parts:
- removed ADDR1: ATF22LV10C, Package_DIP:DIP-24_W7.62mm
- removed AUDIO1, J1, J11, J12: Conn_01x02, Connector_JST:JST_XH_B2B-XH-A_1x02_P2.50mm_Vertical
- removed AUDIO_AMPL2: pam8403, pam8403:pam8403
- removed BankRegister1: 74HC373, Package_DIP:DIP-20_W7.62mm
- removed C1, C10, C20: 1uF, Capacitor_SMD:C_0603_1608Metric
- removed C11, C2: 47uF, Capacitor_SMD:C_0603_1608Metric
- removed C12: 470pF, Capacitor_SMD:C_0603_1608Metric
- removed C13, C14, C21, C23, C25, C4, C5, C6: 100nF, Capacitor_SMD:C_0603_1608Metric
- removed C15: 10µF, Capacitor_SMD:C_0603_1608Metric
- removed C3, C8: 22nF, Capacitor_SMD:C_0603_1608Metric
- removed C7, C9: 10uF, Capacitor_SMD:C_0603_1608Metric
- removed CPU1: W65C816SxP, Package_DIP:DIP-40_W15.24mm
- removed CPU_DB1: 74HC245, Package_DIP:DIP-20_W7.62mm
- removed ETHERNET1: WIZ850IO, AT28C256-15PU:WIZ850IO
- removed Ext0, Ext1: Conn_02x10_Odd_Even, Connector_IDC:IDC-Header_2x10_P2.54mm_Vertical
- removed IC1: DS1818, DS1813-5:TO92127P495H695-3
- removed J5: USB_C_Receptacle_USB2.0_14P, Connector_USB:USB_C_Receptacle_Amphenol_12401610E4-2A_CircularHoles
- removed J7: USB_A, Connector_USB:USB_A_Molex_67643_Horizontal
- removed PWR_PIN1: Conn_02x04_Odd_Even, Connector_PinHeader_2.54mm:PinHeader_2x04_P2.54mm_Vertical
- removed PortA_Ext1, PortC_Ext1, PortD_Ext2: Conn_01x10, Connector_PinHeader_2.54mm:PinHeader_1x10_P2.54mm_Vertical
- removed R1, R16, R19, R2, R25, R26, R27, R28, R4, R8: 10k, Resistor_SMD:R_0603_1608Metric
- removed R17, R3: 4.7k, Resistor_SMD:R_0603_1608Metric
- removed R22, R23: 5.1k, Resistor_SMD:R_0603_1608Metric
- removed R7: 1k, Resistor_SMD:R_0603_1608Metric
- removed RAM1: AS6C4008-55PCN, Package_DIP:DIP-32_W15.24mm
- removed ROM1: AT28LV256, Package_DIP:DIP-28_W15.24mm_Socket
- removed RTC1: DeadOn RTC, Connector_PinHeader_2.54mm:PinHeader_1x07_P2.54mm_Vertical
- removed SDCARD1: Micro_SD_Card, Package_SIP:SIP-9_22.3x3mm_P2.54mm
- removed SERIAL1: SC16C654DBIB64_151, Package_LCC:PLCC-68
- removed SERIAL_C1, SERIAL_D1: Conn_01x04_Pin, Connector_PinHeader_2.54mm:PinHeader_1x04_P2.54mm_Vertical
- removed SID2: SID, Package_DIP:DIP-28_W15.24mm_Socket
- removed SPI_EXT_{3}1: Conn_02x07_Odd_Even, Connector_PinSocket_2.54mm:PinSocket_2x07_P2.54mm_Vertical
- removed SW1: SW_Push, Button_Switch_SMD:SW_Push_1P1T_NO_CK_PTS125Sx73PSMTR
- removed U1, U25: SN74LVC8T245, Package_SO:SSOP-24_3.9x8.7mm_P0.635mm
- removed U2: 2.42OLED, old:DIYMORE.CC
- removed U27: SN74LVC1T45DBV, Package_TO_SOT_SMD:SOT-23-6
- removed U28: 74AHC1G08, Package_TO_SOT_SMD:SOT-23-5
- removed U6, U8, U9: 74HC00, Package_DIP:DIP-14_W7.62mm
- removed UART_USBA1, UART_USBC1: CH340C, Package_SO:SOIC-16_3.9x9.9mm_P1.27mm
- removed VIA1, VIA2: W65C22SxP, Package_DIP:DIP-40_W15.24mm
- removed Y1: TFT680, Oscillator:Oscillator_DIP-14
